File: Hardware/Zombiemaker/Zombiemaker-1.0.sch (KiCad schematic (older format))
At the start: 0 parts

Commit message: WIP commit
squash me after we are finished
Parts:
- added C? (x3): 100nF, Zombiemaker-1.0:C1206, symbol Zombiemaker-1.0-eagle-import:C-EU_C1206K
- added C?: 47µF, Zombiemaker-1.0:C1210, symbol Zombiemaker-1.0-eagle-import:C-EU_C1210K
- added C?: 22µF, Zombiemaker-1.0:C1210, symbol Zombiemaker-1.0-eagle-import:C-EU_C1210K
- added C?: 100nF, Zombiemaker-1.0:C0603, symbol Zombiemaker-1.0-eagle-import:C-EU_C0603K
- added C?: 470uF, Zombiemaker-1.0:ELKO_SMDUD-10X10, symbol Zombiemaker-1.0-eagle-import:ELKOS_UD-10X10
- added H? (x4): MOUNT-PAD-ROUND3.2, Zombiemaker-1.0:3,2-PAD, symbol Zombiemaker-1.0-eagle-import:MOUNT-PAD-ROUND3.2
- added IC?: 7805, Zombiemaker-1.0:78XXS, symbol Zombiemaker-1.0-eagle-import:78XXS
- added L?: XAL6030-332MEB, Zombiemaker-1.0:XAL6030, symbol Zombiemaker-1.0-eagle-import:XAL6030-332MEB
- added R?: 54.9k, Zombiemaker-1.0:R_SMD0603, symbol Zombiemaker-1.0-eagle-import:R-EU_R0603
- added R?: 10.2k, Zombiemaker-1.0:R_SMD0603, symbol Zombiemaker-1.0-eagle-import:R-EU_R0603
- added U?: TPS565208DDCR, Zombiemaker-1.0:DDC0006A_N, symbol Zombiemaker-1.0-eagle-import:TPS565208DDCR
- added U?: LM1117-3.3, Zombiemaker-1.0:SOT223-W, symbol Zombiemaker-1.0-eagle-import:LM1117SOT223-WAVE
- added X? (x4): 22-23-2041, Zombiemaker-1.0:22-23-2041, symbol Zombiemaker-1.0-eagle-import:22-23-2041
Connections:
- net labels added: +12V, +3V3, +5V, GND
- wire segments 0 -> 65
