File: Hardware/Zombiemaker/Zombiemaker-1.0_1.sch (KiCad schematic (older format))
At the start: 18 parts, among them IC1 7805, U2 TPS565208DDCR, U3 LM1117SOT223-WAVE, X1 22-23-2041

Commit message: WIP commit
squash me after we are finished
Connections:
- wire segments 77 -> 76
Changed lines of the file:
@@
 $Descr User 17518 9846
 encoding utf-8
-Sheet 1 5
+Sheet 2 5
 Title ""
 Date ""
@@
 Wire Wire Line
 	6200 1900 6200 800
-Wire Wire Line
-	6200 800  7300 800
-Wire Wire Line
-	7400 800  7300 800
 Connection ~ 6800 1900
 Connection ~ 6200 1900
@@
 $EndComp
 $Comp
-L Zombiemaker-1.0-eagle-import:DINA3_L #FRAME4
-U 2 0 5A848120
-P 12200 9000
-AR Path="/5A848120" Ref="#FRAME4"  Part="2"
-AR Path="/5BBB3611/5A848120" Ref="#FRAME4"  Part="2"
-F 0 "#FRAME4" H 12200 9000 50  0001 C CNN
-F 1 "DINA3_L" H 12200 9000 50  0001 C CNN
-F 2 "" H 12200 9000 50  0001 C CNN
-F 3 "" H 12200 9000 50  0001 C CNN
-	2    12200 9000
-	1    0    0    -1
-$EndComp
-$Comp
 L Zombiemaker-1.0-eagle-import:+12V #P+36
 U 1 0 B49FF82F
@@
 	1    0    0    -1
 $EndComp
+Wire Wire Line
+	6200 800  7400 800
 $EndSCHEMATC
