File: Hardware/Zombiemaker/Zombiemaker-1.0_2.sch (KiCad schematic (older format))
At the start: 71 parts, among them IC2 MCP2200SSOP20, J1 USB_MICRO-BREDUCED_PASTE, U1 ATMEGA2560AU, Y2 CRYSTALSMD-5X3.2-4PAD, Y3 CRYSTALSMD-5X3.2-4PAD

Commit message: WIP commit
squash me after we are finished
Parts:
- removed BLTOUCHD, SERVO, SERVO1, SERVO2, SERVO3: PINHD-1X3, Zombiemaker-1.0:1X03, symbol Zombiemaker-1.0-eagle-import:PINHD-1X3
- removed C35, C43, C46: 100nF, Zombiemaker-1.0:C0603, symbol Zombiemaker-1.0-eagle-import:C-EU_C0603K
- removed FILAMENTERR1, FILAMENTERR2, FILAMENTERR3: MTA02-100, Zombiemaker-1.0:10X02MTA, symbol Zombiemaker-1.0-eagle-import:MTA02-100
- removed JP2: BLTOUCHS, Zombiemaker-1.0:1X02, symbol Zombiemaker-1.0-eagle-import:PINHD-1X2
- removed R100, R101, R34, R84, R95, R96: 10k, Zombiemaker-1.0:R_SMD0603, symbol Zombiemaker-1.0-eagle-import:R-EU_R0603
- renumbered ATX to ATX301, C6 to C301, C5 to C302, C1 to C303, C2 to C304, C4 to C305, C3 to C306, C22 to C307, C7 to C308, C37 to C309, C38 to C310, C14 to C311, C16 to C312, C13 to C313, C12 to C314, C45 to C315, C18 to C316, D6 to D301, D7 to D302, D1 to D303, EXP2 to EXP301, EXP1 to EXP302, I2C to I2C301, IC2 to IC301, ISP1 to ISP301, J1 to J301, JTAG to JTAG301, LED1 to LED301, LED7 to LED302, R42 to R301, R82 to R302, R87 to R303, R88 to R304, R63 to R305, R70 to R306, R98 to R307, R32 to R308, R97 to R309, R33 to R310, R30 to R311, R1 to R312, R99 to R313, R83 to R314, R29 to R315, R4 to R316, R31 to R317, RESET to RESET301, RESETSW to RESETSW301, U$3 to U$301, U1 to U301, UART to UART301, Y3 to Y301, Y2 to Y302
Connections:
- wire segments 354 -> 297
