File: Hardware/Zombiemaker/Zombiemaker-1.0_3.sch (KiCad schematic (older format))
At the start: 57 parts, among them Q1 SI7960, Q2 IRFR430, Q3 MOSFET-NWAVE, Q5 MOSFET-NWAVE, Q7 MOSFET-NWAVE, Q8 MOSFET-NWAVE

Commit message: WIP commit
squash me after we are finished
Parts:
- removed C26, C27, C28, C29: C-EU_C0603K, Zombiemaker-1.0:C0603, symbol Zombiemaker-1.0-eagle-import:C-EU_C0603K
- removed D2, D3, D4, D5: DIODE-SCHOTTKY_, Zombiemaker-1.0:SMA-DIODE, symbol Zombiemaker-1.0-eagle-import:DIODE-SCHOTTKY_
- removed E1-TEMP, E2-TEMP, FAN1, FAN2, FAN3, FAN4, HEATER1, HEATER2, TEMP: MTA02-100, Zombiemaker-1.0:10X02MTA, symbol Zombiemaker-1.0-eagle-import:MTA02-100
- removed HEATBED: MTA04-100, Zombiemaker-1.0:10X04MTA, symbol Zombiemaker-1.0-eagle-import:MTA04-100
- removed LED10, LED2, LED3, LED4, LED5, LED6, LED9: LEDSMT1206, Zombiemaker-1.0:1206, symbol Zombiemaker-1.0-eagle-import:LEDSMT1206
- removed Q1: SI7960, Zombiemaker-1.0:POWERPAK-SO-08-DUAL, symbol Zombiemaker-1.0-eagle-import:SI7960
- removed Q2: IRFR430, Zombiemaker-1.0:DPAK, symbol Zombiemaker-1.0-eagle-import:IRFR430
- removed Q3, Q5, Q7, Q8: MOSFET-NWAVE, Zombiemaker-1.0:SOT23-W, symbol Zombiemaker-1.0-eagle-import:MOSFET-NWAVE
- removed R10, R13, R16, R5, R57, R60, R7: 470, Zombiemaker-1.0:R_SMD0805, symbol Zombiemaker-1.0-eagle-import:R-EU_R0805
- removed R11, R14, R2, R3, R56, R59, R8: 10k, Zombiemaker-1.0:R_SMD0603, symbol Zombiemaker-1.0-eagle-import:R-EU_R0603
- removed R12, R15, R40, R41, R43, R58, R61: 0, Zombiemaker-1.0:R_SMD0603, symbol Zombiemaker-1.0-eagle-import:R-EU_R0603
- removed R64, R65, R66, R67: 4k7, Zombiemaker-1.0:R_SMD0603, symbol Zombiemaker-1.0-eagle-import:R-EU_R0603
- removed R68: 6V/0.5A, Zombiemaker-1.0:1206, symbol Zombiemaker-1.0-eagle-import:PPTC_HALF-AMP
Connections:
- net labels removed: +12V, +5V, FAN1, FAN2, FAN3, FAN4, GND, HEATBED, HEATER1, HEATER2, THERM1, THERM2, THERM3, THERM_BOARD
- wire segments 131 -> 0
