File: Hardware/Zombiemaker/Zombiemaker-1.0_4.sch (KiCad schematic (older format))
At the start: 108 parts, among them T1 -PNP-SOT23-BEC, T2 -PNP-SOT23-BEC, T3 -PNP-SOT23-BEC, T4 -PNP-SOT23-BEC, T5 -PNP-SOT23-BEC, T6 -PNP-SOT23-BEC

Commit message: WIP commit
squash me after we are finished
Parts:
- removed C10, C11, C23, C24, C25, C9: 100nF, Zombiemaker-1.0:C0603, symbol Zombiemaker-1.0-eagle-import:C-EU_C0603K
- removed R17, R19, R21, R23, R25, R27, R44, R46, R48, R50, R52, R54: 1k, Zombiemaker-1.0:R_SMD0603, symbol Zombiemaker-1.0-eagle-import:R-EU_R0603
- removed R18, R22, R26, R45, R49, R53, R76, R77, R78, R79, R80, R81: 0, Zombiemaker-1.0:R_SMD0603, symbol Zombiemaker-1.0-eagle-import:R-EU_R0603
- removed R20, R24, R28, R47, R51, R55: R-EU_R0603, Zombiemaker-1.0:R_SMD0603, symbol Zombiemaker-1.0-eagle-import:R-EU_R0603
- removed T1, T2, T3, T4, T5, T6: -PNP-SOT23-BEC, Zombiemaker-1.0:SOT23-BEC, symbol Zombiemaker-1.0-eagle-import:-PNP-SOT23-BEC
- removed XSTOP, XSTOP1, YSTOP, YSTOP1, ZSTOP, ZSTOP1: MTA03-100, Zombiemaker-1.0:10X03MTA, symbol Zombiemaker-1.0-eagle-import:MTA03-100
- added BLTOUCHD?, SERVO? (x4): PINHD-1X3, Zombiemaker-1.0:1X03, symbol Zombiemaker-1.0-eagle-import:PINHD-1X3
- added D? (x4): DIODE-SCHOTTKY_, Zombiemaker-1.0:SMA-DIODE, symbol Zombiemaker-1.0-eagle-import:DIODE-SCHOTTKY_
- added FAN? (x4), HEATER? (x2): MTA02-100, Zombiemaker-1.0:10X02MTA, symbol Zombiemaker-1.0-eagle-import:MTA02-100
- added HEATBED?: MTA04-100, Zombiemaker-1.0:10X04MTA, symbol Zombiemaker-1.0-eagle-import:MTA04-100
- added JP?: BLTOUCHS, Zombiemaker-1.0:1X02, symbol Zombiemaker-1.0-eagle-import:PINHD-1X2
- added LED? (x7): LEDSMT1206, Zombiemaker-1.0:1206, symbol Zombiemaker-1.0-eagle-import:LEDSMT1206
- added Q? (x4): MOSFET-NWAVE, Zombiemaker-1.0:SOT23-W, symbol Zombiemaker-1.0-eagle-import:MOSFET-NWAVE
- added Q?: IRFR430, Zombiemaker-1.0:DPAK, symbol Zombiemaker-1.0-eagle-import:IRFR430
- added Q? (x2): SI7960, Zombiemaker-1.0:POWERPAK-SO-08-DUAL, symbol Zombiemaker-1.0-eagle-import:SI7960
- added R? (x7): 10k, Zombiemaker-1.0:R_SMD0603, symbol Zombiemaker-1.0-eagle-import:R-EU_R0603
- added R? (x7): 470, Zombiemaker-1.0:R_SMD0805, symbol Zombiemaker-1.0-eagle-import:R-EU_R0805
- added R? (x7): 0, Zombiemaker-1.0:R_SMD0603, symbol Zombiemaker-1.0-eagle-import:R-EU_R0603
Connections:
- net labels added: BLTOUCH, FAN1, FAN2, FAN3, FAN4, HEATBED, HEATER1, HEATER2, SERVO1, SERVO2, SERVO3, SERVO4, ZMIN
- net labels removed: XSTOP, XSTOP1, YSTOP, YSTOP1, ZSTOP, ZSTOP1
